File: b_nahl_v1/b_nahl_v1.kicad_pcb (KiCad board)
At the start: 2 copper layers, 14 parts

Commit message: Version finale
Parts:
- removed R3, R4: 4.7k, Resistor_THT:R_Axial_DIN0207_L6.3mm_D2.5mm_P7.62mm_Horizontal
- added H1: MountingHole, MountingHole:MountingHole_3.2mm_M3, F.Cu at (104.0, 62.5)
- added H2: MountingHole, MountingHole:MountingHole_3.2mm_M3, F.Cu at (168.5, 62.5)
- added H3: MountingHole, MountingHole:MountingHole_3.2mm_M3, F.Cu at (168.5, 113.0)
- added H4: MountingHole, MountingHole:MountingHole_3.2mm_M3, F.Cu at (104.0, 113.0)
- moved S7V8F3 62.8 mm to (116.5, 64.0)
- moved DHT22 53.6 mm to (153.0, 111.0), turned to 180 degrees
- moved SHT20 48.4 mm to (147.0, 64.0)
- moved TSL2561 48.4 mm to (153.5, 64.0)
- moved Nano_33_BLE1 48.0 mm to (140.0, 64.5)
- moved R1 39.9 mm to (125.3, 103.0), turned to 180 degrees
- moved DS18B21 39.6 mm to (146.5, 111.0), turned to 180 degrees
- moved R2 32.4 mm to (117.7, 107.0)
- moved HX711 30.0 mm to (159.5, 111.0), turned to 180 degrees
- moved DS18B20 25.6 mm to (140.0, 111.0), turned to 180 degrees
- moved A1 17.8 mm to (105.0, 77.0)
- moved Entree1 10.6 mm to (112.0, 109.0), turned to 180 degrees
- renumbered DS18B1 to DS18B21
Connections:
- A1 pad 3V3: 3V3 -> VCC 3V3
- A1 pad D1: Cout -> unconnected-(A1-PadD1)
- A1 pad D11: Net-(A1-D11/SDA) -> SDA
- A1 pad D12: Net-(A1-D12/SCL) -> SCL
- A1 pad D14: unconnected-(A1-D14/TX-PadD14) -> TX
- A1 pad D3: D3 -> Cout
- A1 pad D4: SHDN -> SCK
- A1 pad D6: SCK -> SHDN
- DHT22 pad 3: D2 -> unconnected-(DHT22-Pad3)
- DHT22 pad 4: unconnected-(DHT22-Pad4) -> D2
- DS18B20 pad 3: D0 -> unconnected-(DS18B20-Pad3)
- DS18B20 pad 4: unconnected-(DS18B20-Pad4) -> D0
- DS18B21 pad 3: D3 -> unconnected-(DS18B21-Pad3)
- DS18B21 pad 4: unconnected-(DS18B1-Pad4) -> D0
- Nano_33_BLE1 pad 3: unconnected-(Nano_33_BLE1-Pad3) -> TX
- SHT20 pad 3: SDA -> SCL
- SHT20 pad 4: SCL -> SDA
- TSL2561 pad 3: SDA -> SCL
- TSL2561 pad 4: SCL -> SDA
Routing:
- net VCC 3V3: track 0.00 -> 170.4 mm
- net SHDN: track 0.00 -> 46.8 mm, vias 0 -> 2
- net VOUT: track 0.00 -> 26.0 mm
- net SCL: track 0.00 -> 19.7 mm
- net D0: track 0.00 -> 17.0 mm
- net Cout: track 0.00 -> 16.2 mm
- net SDA: track 0.00 -> 15.2 mm
- net ADC: track 0.00 -> 11.9 mm
- net SCK: track 0.00 -> 11.6 mm
- net TX: track 0.00 -> 11.0 mm
- net D2: track 0.00 -> 10.2 mm
- net RX: track 0.00 -> 6.64 mm
- net Ve: track 0.00 -> 5.69 mm
- added copper zone on B.Cu, net GND
Other:
- board outline added: 71.5 x 57.5 mm
- board text added: "B-NAHL"
